File: qualification/class-b/usb-uart/kicad/usb_uart.kicad_pcb (KiCad board)
At the start: 4 copper layers, 50.4 x 38.3 mm, 40 parts, among them J1 12401610E4#2A, J2 UART1, J3 FLOW1, J4 RS485, U1 CH342F, U2 LDO, U3 THVD1450D

Commit message: SYN-66 - Route the board again with the merged Synth tools
All the tool PRs this board needed are merged (#154, #162, #173, #175,
#176, #197, #198, #200), so it is exported again with Synth main
9c0fc2c. With #200 the pads of rotated parts turn with the part: D8's
lands now stand vertical, and FreeRouting finds another route (276
segments, 45 vias, 585 mm). KiCad DRC is 0 errors and 0 unconnected,
also after a re-save, and the release gate passes.

The schematic now carries the declared net names and the net class
rules in the project file use the PCB's names. Images, STEP file,
reports and hashes are regenerated and the docs say what changed.

Signed-off-by: nyagamunene <stevenyaga2014@gmail.com>
Routing:
- net RS485_B_BUS: track 29.7 -> 31.3 mm
- net RS485_A_BUS: track 17.0 -> 18.0 mm
- net GND: vias 22 -> 23
