File: qualification/class-b/usb-uart/kicad/usb_uart.kicad_sch (KiCad schematic)
At the start: 40 parts, among them J1 12401610E4#2A, J2 UART1, J3 FLOW1, J4 RS485, U1 CH342F, U2 LDO, U3 THVD1450D

Commit message: SYN-66 - Route the board again with the merged Synth tools
All the tool PRs this board needed are merged (#154, #162, #173, #175,
#176, #197, #198, #200), so it is exported again with Synth main
9c0fc2c. With #200 the pads of rotated parts turn with the part: D8's
lands now stand vertical, and FreeRouting finds another route (276
segments, 45 vias, 585 mm). KiCad DRC is 0 errors and 0 unconnected,
also after a re-save, and the release gate passes.

The schematic now carries the declared net names and the net class
rules in the project file use the PCB's names. Images, STEP file,
reports and hashes are regenerated and the docs say what changed.

Signed-off-by: nyagamunene <stevenyaga2014@gmail.com>
Connections:
- net CTS0 renamed CTS0_LOW
- net CTS1 renamed CTS1_MCU
- net D+ renamed USB_DP
- net D- renamed USB_DN
- net DTR0_TNOW0 renamed TNOW0
- net DTR1_TNOW1 renamed DTR1
- net P2 renamed RS485_A_BUS
- net RI0 renamed MODEM_IDLE
- net RX renamed RXD1_MCU
- net RX_U1 renamed RXD0
- net TX renamed TXD1
- net TX_U1 renamed TXD0
Changed lines of the file:
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@@
 		(pts
 			(xy 520.7 35.56)
-			(xy 520.7 81.28)
+			(xy 523.24 35.56)
 		)
 		(stroke
@@
 	(wire
 		(pts
-			(xy 520.7 81.28)
-			(xy 483.87 81.28)
+			(xy 523.24 35.56)
+			(xy 523.24 111.76)
 		)
 		(stroke
@@
 	(wire
 		(pts
-			(xy 483.87 81.28)
-			(xy 483.87 96.52)
+			(xy 523.24 111.76)
+			(xy 486.41 111.76)
 		)
 		(stroke
@@
 	(wire
 		(pts
-			(xy 483.87 96.52)
+			(xy 486.41 111.76)
 			(xy 486.41 96.52)
 		)
@@
 		(pts
 			(xy 494.03 96.52)
-			(xy 499.11 96.52)
+			(xy 496.57 96.52)
 		)
 		(stroke
@@
 	(wire
 		(pts
-			(xy 499.11 96.52)
-			(xy 499.11 49.53)
+			(xy 496.57 96.52)
+			(xy 496.57 22.86)
 		)
 		(stroke
@@
 	(wire
 		(pts
-			(xy 499.11 49.53)
-			(xy 458.47 49.53)
+			(xy 496.57 22.86)
+			(xy 462.28 22.86)
 		)
 		(stroke
@@
 	(wire
 		(pts
-			(xy 458.47 49.53)
-			(xy 458.47 38.1)
+			(xy 462.28 22.86)
+			(xy 462.28 38.1)
 		)
 		(stroke
@@
 	(wire
 		(pts
-			(xy 458.47 38.1)
+			(xy 462.28 38.1)
 			(xy 464.82 38.1)
 		)
@@
 	(wire
 		(pts
-			(xy 494.03 96.52)
 			(xy 496.57 96.52)
+			(xy 496.57 81.28)
 		)
 		(stroke
@@
 	(wire
 		(pts
-			(xy 496.57 96.52)
-			(xy 496.57 114.3)
+			(xy 496.57 81.28)
+			(xy 528.32 81.28)
 		)
 		(stroke
@@
 	(wire
 		(pts
-			(xy 496.57 114.3)
-			(xy 530.86 114.3)
+			(xy 528.32 81.28)
+			(xy 528.32 99.06)
 		)
 		(stroke
@@
 	(wire
 		(pts
-			(xy 530.86 114.3)
+			(xy 528.32 99.06)
 			(xy 530.86 99.06)
 		)
@@
 		(color 0 0 0 0)
 	)
+	(junction
+		(at 496.57 96.52)
+		(diameter 0)
+		(color 0 0 0 0)
+	)
 	(wire
 		(pts
@@
 	)
 	(label
-		"D+"
+		"USB_DP"
 		(at 55.88 48.26 0)
 		(effects
@@
 	)
 	(label
-		"D+"
+		"USB_DP"
 		(at 55.88 50.8 0)
 		(effects
@@
 	)
 	(label
-		"D+"
+		"USB_DP"
 		(at 106.68 33.02 180)
 		(effects
@@
 	)
 	(label
-		"D+"
+		"USB_DP"
 		(at 260.35 49.53 180)
 		(effects
@@
 	)
 	(label
-		"D-"
+		"USB_DN"
 		(at 55.88 43.18 0)
 		(effects
@@
 	)
 	(label
-		"D-"
+		"USB_DN"
 		(at 55.88 45.72 0)
 		(effects
@@
 	)
 	(label
-		"D-"
+		"USB_DN"
 		(at 142.24 33.02 0)
 		(effects
@@
 	)
 	(label
-		"D-"
+		"USB_DN"
 		(at 260.35 52.07 180)
 		(effects
@@
 	)
 	(label
-		"TX"
+		"TXD1"
 		(at 293.37 49.53 0)
 		(effects
@@
 	)
 	(label
-		"TX"
+		"TXD1"
 		(at 419.1 30.48 180)
 		(effects
@@
 	)
 	(label
-		"TX"
+		"TXD1"
 		(at 109.22 173.99 0)
 		(effects
@@
 	)
 	(label
-		"RX"
+		"RXD1_MCU"
 		(at 402.59 33.02 180)
 		(effects
@@
 	)
 	(label
-		"RX"
+		"RXD1_MCU"
 		(at 260.35 64.77 180)
 		(effects
@@
 	)
 	(label
-		"DTR1_TNOW1"
+		"DTR1"
 		(at 293.37 52.07 0)
 		(effects
@@
 	)
 	(label
-		"DTR1_TNOW1"
+		"DTR1"
 		(at 419.1 58.42 180)
 		(effects
@@
 	)
 	(label
-		"CTS1"
+		"CTS1_MCU"
 		(at 402.59 63.5 180)
 		(effects
@@
 	)
 	(label
-		"CTS1"
+		"CTS1_MCU"
 		(at 260.35 62.23 180)
 		(effects
@@
 	)
 	(label
-		"TX_U1"
+		"TXD0"
 		(at 293.37 57.15 0)
 		(effects
@@
 	)
 	(label
-		"TX_U1"
+		"TXD0"
 		(at 495.3 43.18 180)
 		(effects
@@
 	)
 	(label
-		"TX_U1"
+		"TXD0"
 		(at 76.2 173.99 0)
 		(effects
@@
 	)
 	(label
-		"RX_U1"
+		"RXD0"
 		(at 260.35 77.47 180)
 		(effects
@@
 	)
 	(label
-		"RX_U1"
+		"RXD0"
 		(at 495.3 33.02 180)
 		(effects
@@
 	)
 	(label
-		"DTR0_TNOW0"
+		"TNOW0"
 		(at 293.37 59.69 0)
 		(effects
@@
 	)
 	(label
-		"DTR0_TNOW0"
+		"TNOW0"
 		(at 495.3 38.1 180)
 		(effects
@@
 	)
 	(label
-		"DTR0_TNOW0"
+		"TNOW0"
 		(at 495.3 35.56 180)
 		(effects
@@
 	)
 	(label
-		"DTR0_TNOW0"
+		"TNOW0"
 		(at 544.83 38.1 180)
 		(effects
@@
 	)
 	(label
-		"P2"
+		"RS485_A_BUS"
 		(at 478.79 96.52 0)
 		(effects
@@
 	)
 	(label
-		"P2"
+		"RS485_A_BUS"
 		(at 459.74 35.56 180)
 		(effects
@@
 	)
 	(label
-		"P2"
+		"RS485_A_BUS"
 		(at 495.3 92.71 180)
 		(effects
@@
 	)
 	(label
-		"P2"
+		"RS485_A_BUS"
 		(at 558.8 77.47 0)
 		(effects
@@
 	)
 	(label
-		"RI0"
+		"MODEM_IDLE"
 		(at 260.35 46.99 180)
 		(effects
@@
 	)
 	(label
-		"RI0"
+		"MODEM_IDLE"
 		(at 242.57 43.18 0)
 		(effects
@@
 	)
 	(label
-		"RI0"
+		"MODEM_IDLE"
 		(at 260.35 72.39 180)
 		(effects
@@
 	)
 	(label
-		"RI0"
+		"MODEM_IDLE"
 		(at 260.35 82.55 180)
 		(effects
@@
 	)
 	(label
-		"RI0"
+		"MODEM_IDLE"
 		(at 260.35 69.85 180)
 		(effects
@@
 	)
 	(label
-		"RI0"
+		"MODEM_IDLE"
 		(at 260.35 80.01 180)
 		(effects
@@
 	)
 	(label
-		"RI0"
+		"MODEM_IDLE"
 		(at 260.35 67.31 180)
 		(effects
@@
 	)
 	(label
-		"CTS0"
+		"CTS0_LOW"
 		(at 260.35 74.93 180)
 		(effects
@@
 	)
 	(label
-		"CTS0"
+		"CTS0_LOW"
 		(at 224.79 78.74 180)
 		(effects
