File: qualification/class-b/ble_node/kicad/ble_node.kicad_sch (KiCad schematic)
At the start: 28 parts, among them J1 TYPE-C-31-M-12, U1 nRF52840-QIAA, U2 BME680, X1 32 MHz

Commit message: fix: address PR review - restructure as qualification boards, fix RTD topology, USB ESD, BME280 (SYN-365)
Changes:
- Move from examples/ to qualification/class-b/<board>/ with README, SHA256SUMS, qualification.json
- Fix RTD amplifier: non-inverting gain stage (1+R2/R1=11x) instead of inverting
- Fix USB ESD: separate D_ESD_DP and D_ESD_DN diodes instead of shorting D+/D-
- Add BME280 part to registry (issue specifies BME280, not BME680)
- Add i2c_sda/i2c_scl capabilities to nrf52840 p0_06/p0_08
- Fix balun_2g4 footprint to real KiCad part
- Re-route BLE node: 0 unconnected pads (manual via-in-pad escape)
- Add DRC/ERC reports, SHA256SUMS, qualification.json for both boards
- Remove silkscreen labels, add USB-C 3D model reference
Parts:
- removed D_ESD: (no value), Diode_SMD:D_SOD-323, symbol Device:D_TVS
- added D_ESD_DN, D_ESD_DP: (no value), Diode_SMD:D_SOD-323, symbol Device:D_TVS
- U2: value BME680 -> BME280; symbol Sensor:BME680 -> Sensor:BME280; LCSC (none) -> C92489; MPN (none) -> BME280
Connections:
- net P0_26 is gone; now on net SDA: J_SWD.2 (Pin_2), U1.G1 (p0_26)
- net P0_27 is gone; now on net SCL: J_SWD.3 (Pin_3), U1.H2 (p0_27)
- net DP: now also D_ESD_DP.1 (A1); no longer J1.A7 (D-)
- net GND: now also D_ESD_DN.2 (A2), D_ESD_DP.2 (A2)
- net SCL: no longer R_I2C_SCL.1, U1.N1 (scl), U2.4 (SCK)
- net SDA: no longer R_I2C_SDA.1, U1.L1 (sda), U2.3 (SDI)
- new net DN: D_ESD_DN.1 (A1), J1.A7 (D-)
- new net RX: R_I2C_SCL.1, U1.N1 (p0_08), U2.4 (SCK)
- new net TX: R_I2C_SDA.1, U1.L1 (p0_06), U2.3 (SDI)
Other:
- note added: "BME280 ENVIRONMENT SENSOR"
- note added: "BME280: temp, humidity, pressure (I2C, addr 0x76)."
- note removed: "BME680 ENVIRONMENT SENSOR"
- note removed: "BME680: temp, humidity, pressure, gas/VOC."
- moved on the sheet: ANT1, B1, C_ANT, C_DEC1, C_DEC2, C_LDO_IN, C_LDO_OUT, C_MATCH1, C_RESET, C_SENS, C_VBUS, C_XTAL1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
